File: pcb_files/hexapad.kicad_pcb (KiCad board)
At the start: 2 copper layers, 210 x 209.7 mm, 12 parts, among them SW1 SW_Push, SW2 SW_Push, U1 SeeeduinoXIAO, U2 VL53L0X

Commit message: update pcb and sysex
Parts:
- C1: value 100n -> 100nF
- C2: value 4.7u -> 4.7uF
- R1, R2, R3, R4: value 2k -> 2K
- R5: value 20 -> 20K
Changed lines of the file:
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@@
       (disableapertmacros false)
       (usegerberextensions true)
-      (usegerberattributes false)
+      (usegerberattributes true)
       (usegerberadvancedattributes false)
       (creategerberjobfile false)
@@
       (drillshape 0)
       (scaleselection 1)
-      (outputdirectory "gerbers_hexapad")
+      (outputdirectory "CPL_hexapad")
     )
   )
@@
       (effects (font (size 1 1) (thickness 0.15)) (justify mirror))
     )
-    (fp_text value "2k" (at 0 -1.65) (layer "B.Fab")
+    (fp_text value "2K" (at 0 -1.65) (layer "B.Fab")
       (effects (font (size 1 1) (thickness 0.15)) (justify mirror))
     )
@@
       (effects (font (size 1 1) (thickness 0.15)) (justify mirror))
     )
-    (fp_text value "20" (at 0 -1.65) (layer "B.Fab")
+    (fp_text value "20K" (at 0 -1.65) (layer "B.Fab")
       (effects (font (size 1 1) (thickness 0.15)) (justify mirror))
     )
@@
       (effects (font (size 1 1) (thickness 0.15)) (justify mirror))
     )
-    (fp_text value "2k" (at 0 -1.65) (layer "B.Fab")
+    (fp_text value "2K" (at 0 -1.65) (layer "B.Fab")
       (effects (font (size 1 1) (thickness 0.15)) (justify mirror))
     )
@@
       (effects (font (size 1 1) (thickness 0.15)) (justify mirror))
     )
-    (fp_text value "2k" (at 0 -1.65) (layer "B.Fab")
+    (fp_text value "2K" (at 0 -1.65) (layer "B.Fab")
       (effects (font (size 1 1) (thickness 0.15)) (justify mirror))
     )
@@
       (effects (font (size 1 1) (thickness 0.15)) (justify mirror))
     )
-    (fp_text value "4.7u" (at -0.05 1.71) (layer "B.Fab")
+    (fp_text value "4.7uF" (at -0.05 1.71) (layer "B.Fab")
       (effects (font (size 1 1) (thickness 0.15)) (justify mirror))
     )
@@
       (effects (font (size 1 1) (thickness 0.15)) (justify mirror))
     )
-    (fp_text value "100n" (at 0 -1.16) (layer "B.Fab")
+    (fp_text value "100nF" (at 0 -1.16) (layer "B.Fab")
       (effects (font (size 1 1) (thickness 0.15)) (justify mirror))
     )
@@
       (effects (font (size 1 1) (thickness 0.15)) (justify mirror))
     )
-    (fp_text value "2k" (at 0 -1.65) (layer "B.Fab")
+    (fp_text value "2K" (at 0 -1.65) (layer "B.Fab")
       (effects (font (size 1 1) (thickness 0.15)) (justify mirror))
     )
